File: pcb_schematics/_autosave-pcb_schematics.kicad_sch (KiCad schematic)
At the start: 71 parts, among them J1 CUE_SJ1-352XNG, J2 Conn_01x01_Pin, J3 Conn_01x05, J4 Conn_01x05, J5 Conn_01x05, SW1 SW_Push, U1 RPi_Pico_TH, U2 RDA5807M_Module, U3 LM386, U4 LM386

Commit message: compeltes PCB
Only the DRC has a couple errors
Parts:
- TP1, TP10, TP11, TP12, TP13, TP14, TP15, TP16, TP17, TP18, TP19, TP2, TP3, TP4, TP5, TP6, TP7, TP8, TP9: footprint TestPoint:TestPoint_Loop_D2.50mm_Drill1.0mm -> TestPoint:TestPoint_Keystone_5000-5004_Miniature
Changed lines of the file:
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@@
       (effects (font (size 1.27 1.27)) (justify right))
     )
-    (property "Footprint" "TestPoint:TestPoint_Loop_D2.50mm_Drill1.0mm" (at 200.66 86.36 0)
+    (property "Footprint" "TestPoint:TestPoint_Keystone_5000-5004_Miniature" (at 200.66 86.36 0)
       (effects (font (size 1.27 1.27)) hide)
     )
@@
       (effects (font (size 1.27 1.27)) (justify right))
     )
-    (property "Footprint" "TestPoint:TestPoint_Loop_D2.50mm_Drill1.0mm" (at 170.18 110.49 0)
+    (property "Footprint" "TestPoint:TestPoint_Keystone_5000-5004_Miniature" (at 170.18 110.49 0)
       (effects (font (size 1.27 1.27)) hide)
     )
@@
       (effects (font (size 1.27 1.27)) (justify left))
     )
-    (property "Footprint" "TestPoint:TestPoint_Loop_D2.50mm_Drill1.0mm" (at 38.1 116.84 0)
+    (property "Footprint" "TestPoint:TestPoint_Keystone_5000-5004_Miniature" (at 38.1 116.84 0)
       (effects (font (size 1.27 1.27)) hide)
     )
@@
       (effects (font (size 1.27 1.27)) (justify left))
     )
-    (property "Footprint" "TestPoint:TestPoint_Loop_D2.50mm_Drill1.0mm" (at 203.2 78.74 0)
+    (property "Footprint" "TestPoint:TestPoint_Keystone_5000-5004_Miniature" (at 203.2 78.74 0)
       (effects (font (size 1.27 1.27)) hide)
     )
@@
       (effects (font (size 1.27 1.27)) (justify left))
     )
-    (property "Footprint" "TestPoint:TestPoint_Loop_D2.50mm_Drill1.0mm" (at 80.01 76.2 0)
+    (property "Footprint" "TestPoint:TestPoint_Keystone_5000-5004_Miniature" (at 80.01 76.2 0)
       (effects (font (size 1.27 1.27)) hide)
     )
@@
       (effects (font (size 1.27 1.27)) (justify right))
     )
-    (property "Footprint" "TestPoint:TestPoint_Loop_D2.50mm_Drill1.0mm" (at 226.06 31.75 0)
+    (property "Footprint" "TestPoint:TestPoint_Keystone_5000-5004_Miniature" (at 226.06 31.75 0)
       (effects (font (size 1.27 1.27)) hide)
     )
@@
       (effects (font (size 1.27 1.27)) (justify left))
     )
-    (property "Footprint" "TestPoint:TestPoint_Loop_D2.50mm_Drill1.0mm" (at 80.01 81.28 0)
+    (property "Footprint" "TestPoint:TestPoint_Keystone_5000-5004_Miniature" (at 80.01 81.28 0)
       (effects (font (size 1.27 1.27)) hide)
     )
@@
       (effects (font (size 1.27 1.27)) (justify left))
     )
-    (property "Footprint" "TestPoint:TestPoint_Loop_D2.50mm_Drill1.0mm" (at 124.46 95.25 0)
+    (property "Footprint" "TestPoint:TestPoint_Keystone_5000-5004_Miniature" (at 124.46 95.25 0)
       (effects (font (size 1.27 1.27)) hide)
     )
@@
       (effects (font (size 1.27 1.27)) (justify left))
     )
-    (property "Footprint" "TestPoint:TestPoint_Loop_D2.50mm_Drill1.0mm" (at 80.01 78.74 0)
+    (property "Footprint" "TestPoint:TestPoint_Keystone_5000-5004_Miniature" (at 80.01 78.74 0)
       (effects (font (size 1.27 1.27)) hide)
     )
@@
       (effects (font (size 1.27 1.27)) (justify right))
     )
-    (property "Footprint" "TestPoint:TestPoint_Loop_D2.50mm_Drill1.0mm" (at 224.79 88.9 0)
+    (property "Footprint" "TestPoint:TestPoint_Keystone_5000-5004_Miniature" (at 224.79 88.9 0)
       (effects (font (size 1.27 1.27)) hide)
     )
@@
       (effects (font (size 1.27 1.27)) (justify left))
     )
-    (property "Footprint" "TestPoint:TestPoint_Loop_D2.50mm_Drill1.0mm" (at 106.68 100.33 0)
+    (property "Footprint" "TestPoint:TestPoint_Keystone_5000-5004_Miniature" (at 106.68 100.33 0)
       (effects (font (size 1.27 1.27)) hide)
     )
@@
       (effects (font (size 1.27 1.27)) (justify left))
     )
-    (property "Footprint" "TestPoint:TestPoint_Loop_D2.50mm_Drill1.0mm" (at 123.19 160.02 0)
+    (property "Footprint" "TestPoint:TestPoint_Keystone_5000-5004_Miniature" (at 123.19 160.02 0)
       (effects (font (size 1.27 1.27)) hide)
     )
@@
       (effects (font (size 1.27 1.27)) (justify right))
     )
-    (property "Footprint" "TestPoint:TestPoint_Loop_D2.50mm_Drill1.0mm" (at 113.03 176.53 0)
+    (property "Footprint" "TestPoint:TestPoint_Keystone_5000-5004_Miniature" (at 113.03 176.53 0)
       (effects (font (size 1.27 1.27)) hide)
     )
@@
       (effects (font (size 1.27 1.27)) (justify right))
     )
-    (property "Footprint" "TestPoint:TestPoint_Loop_D2.50mm_Drill1.0mm" (at 45.72 175.26 0)
+    (property "Footprint" "TestPoint:TestPoint_Keystone_5000-5004_Miniature" (at 45.72 175.26 0)
       (effects (font (size 1.27 1.27)) hide)
     )
@@
       (effects (font (size 1.27 1.27)) (justify right))
     )
-    (property "Footprint" "TestPoint:TestPoint_Loop_D2.50mm_Drill1.0mm" (at 29.21 134.62 0)
+    (property "Footprint" "TestPoint:TestPoint_Keystone_5000-5004_Miniature" (at 29.21 134.62 0)
       (effects (font (size 1.27 1.27)) hide)
     )
@@
       (effects (font (size 1.27 1.27)) (justify left))
     )
-    (property "Footprint" "TestPoint:TestPoint_Loop_D2.50mm_Drill1.0mm" (at 205.74 20.32 0)
+    (property "Footprint" "TestPoint:TestPoint_Keystone_5000-5004_Miniature" (at 205.74 20.32 0)
       (effects (font (size 1.27 1.27)) hide)
     )
@@
       (effects (font (size 1.27 1.27)) (justify left))
     )
-    (property "Footprint" "TestPoint:TestPoint_Loop_D2.50mm_Drill1.0mm" (at 184.15 105.41 0)
+    (property "Footprint" "TestPoint:TestPoint_Keystone_5000-5004_Miniature" (at 184.15 105.41 0)
       (effects (font (size 1.27 1.27)) hide)
     )
@@
       (effects (font (size 1.27 1.27)) (justify right))
     )
-    (property "Footprint" "TestPoint:TestPoint_Loop_D2.50mm_Drill1.0mm" (at 201.93 29.21 0)
+    (property "Footprint" "TestPoint:TestPoint_Keystone_5000-5004_Miniature" (at 201.93 29.21 0)
       (effects (font (size 1.27 1.27)) hide)
     )
@@
       (effects (font (size 1.27 1.27)) (justify left))
     )
-    (property "Footprint" "TestPoint:TestPoint_Loop_D2.50mm_Drill1.0mm" (at 57.15 158.75 0)
-      (effects (font (size 1.27 1.27)) hide)
-    )
+    (property "Footprint" "TestPoint:TestPoint_Keystone_5000-5004_Miniature" (at 57.15 158.75 0)
+      (effects (font (size 1.27 1.27)) hide)
+    )
