File: pcb_schematics/pcb_schematics.kicad_sch (KiCad schematic)
At the start: 30 parts, among them J1 CUE_SJ1-352XNG, J2 Conn_01x01_Pin, SW1 SW_Push, SW2 Bourns PEC11R, SW7 Bourns PEC11R, SW8 Bourns PEC11R, U1 RPi_Pico_TH, U2 RDA5807M_Module, U3 LM386, U4 LM386

Commit message: Pcb (#1)
* Converted to connectors

* Updates PCb according to ROB's feedback

Added PCb layour according to the discussion with butoons and display on top and display below using front copper. Added Radio module using back copper. Speakers left to set up using back copper.

* compeltes PCB

Only the DRC has a couple errors

* Updates footprints in schematic

* Fixes errors in DRC

Adds SMD capacitors too

* Runs DRC and ERC again

* Accomodating usb cable

* Revision 3

Changed the amplifier and the rotary encoder schemtic. Needs work on pcb

* completes third version of PCB

* fixed issues mentioned by rob and brent

Fix iteration 1

* made changes based on changes requested

Fix iteration 2

* Submitted to JLCPCB

Modification with pcb_schematics being the final version.
Parts:
- removed C1, C2: 10 µF, Capacitor_THT:CP_Radial_D5.0mm_P2.00mm, symbol Device:C
- removed C3, C6: 250 µF, symbol Device:C_Small
- removed R3, R4: 10Ω, Resistor_THT:R_Axial_DIN0207_L6.3mm_D2.5mm_P10.16mm_Horizontal, symbol Device:R_US
- removed SW2, SW7, SW8: Bourns PEC11R, Rotary_Encoder:RotaryEncoder_Alps_EC12E-Switch_Vertical_H20mm, symbol ECE:Bourns PEC11R
- added C1, C10, C11, C14, C2, C9: 0.01 µF, Capacitor_THT:C_Axial_L3.8mm_D2.6mm_P7.50mm_Horizontal, symbol Device:C_Small
- added C12, C13: 0.1 µF, Capacitor_THT:C_Axial_L3.8mm_D2.6mm_P7.50mm_Horizontal, symbol Device:C_Small
- added C15, C16, C3, C6: 470 µF, Capacitor_THT:CP_Radial_D6.3mm_P2.50mm, symbol Device:C_Polarized_US
- added H1, H2, H3, H4: MountingHole, MountingHole:MountingHole_3.2mm_M3, symbol Mechanical:MountingHole
- added J3, J4, J5: Conn_01x05, Connector_PinHeader_2.54mm:PinHeader_1x05_P2.54mm_Vertical, symbol Connector_Generic:Conn_01x05
- added R10, R5, R6, R9: 10Ω, Resistor_THT:R_Axial_DIN0207_L6.3mm_D2.5mm_P10.16mm_Horizontal, symbol Device:R_US
- added R3, R4: 10 k, Resistor_THT:R_Axial_DIN0207_L6.3mm_D2.5mm_P10.16mm_Horizontal, symbol Device:R
- added R7, R8, R_Pullup1, R_Pullup2, R_Pullup4, R_Pullup5, R_Pullup6, R_Pullup7: 10kΩ, Resistor_THT:R_Axial_DIN0207_L6.3mm_D2.5mm_P10.16mm_Horizontal, symbol Device:R_US
- added TP1, TP10, TP11, TP12, TP13, TP14, TP15, TP16, TP17, TP18, TP19, TP2, TP3, TP4, TP5, TP6, TP7, TP8, TP9: TestPoint, TestPoint:TestPoint_Keystone_5000-5004_Miniature, symbol Connector:TestPoint
- C4, C5: footprint (none) -> Capacitor_THT:C_Axial_L3.8mm_D2.6mm_P7.50mm_Horizontal
- C7, C8: value 0.05 µF -> 0.1 µF; footprint (none) -> Capacitor_SMD:C_0603_1608Metric
- J1: footprint ECE:CUE_SJ1-352XNG -> Connector_PinHeader_2.54mm:PinHeader_1x05_P2.54mm_Vertical
- J2: footprint Connector:Banana_Jack_1Pin -> Connector_Pin:Pin_D1.0mm_L10.0mm_LooseFit
- LS1, LS2: footprint ECE:CUE_CMA-4544PF-W -> TerminalBlock_Phoenix:TerminalBlock_Phoenix_MKDS-1,5-2_1x02_P5.00mm_Horizontal
- RV1, RV2: footprint ECE:Bourns_PTV09_Horiz -> Connector_PinHeader_2.54mm:PinHeader_1x03_P2.54mm_Vertical
- R_Pullup3: value 2kΩ -> 10kΩ
- SW1: footprint Button_Switch_THT:Push_E-Switch_KS01Q01 -> Connector_PinHeader_2.54mm:PinHeader_1x02_P2.54mm_Vertical
Connections:
- net +5V: now also C7.2, C8.2, U3.6 (V+), U4.6 (V+), C12.2, C13.2
- net 3V3: now also R_Pullup1.2, R_Pullup2.2, R_Pullup4.2, R_Pullup5.2, R_Pullup6.2, R_Pullup7.2; no longer U3.6 (V+), U4.6 (V+)
- net CS: now also TP2.1
- net GND: now also C7.1, C8.1, C1.2, C10.1, C11.1, C12.1, C13.1, C14.1, C2.2, C9.2, J3.2 (Pin_2), J3.3 (Pin_3), J4.2 (Pin_2), J4.3 (Pin_3), J5.2 (Pin_2), J5.3 (Pin_3)
- net I2CSCK: now also TP5.1
- net I2CTX: now also TP4.1
- net LOUT: now also J1.2 (Tip), TP10.1; no longer C7.1, J1.4 (Tip_Switch)
- net LSpeaker: now also J1.5 (Ring_Switch), R3.2; no longer J1.3 (Tip), RV1.1
- net ROUT: now also J1.3 (Tip), TP11.1; no longer C8.1, J1.5 (Ring_Switch)
- net RSpeaker: now also J1.4 (Tip_Switch), R4.1; no longer J1.2 (Tip), RV2.1
- net SCK: now also TP1.1
- net SDA: now also TP3.1
- net SW2: now also U1.2 (GP1), J4.4 (Pin_4); no longer U1.4 (GP2)
- net SW3: now also U1.31 (GP26/ADC0), J3.4 (Pin_4); no longer U1.6 (GP4)
- net SW4: now also U1.7 (GP5), J5.4 (Pin_4); no longer U1.9 (GP6)
- net at RV1.2: now also C15.1, TP7.1; no longer U3.3 (+)
- net at LS2.1: now also C3.2
- net at C5.1, U3.5: now also C6.1, TP8.1
- net at LS1.1: now also C6.2
- net ROT2B: now reaches U1.10 (GP7)
- net ROT2B: now also C11.2, R8.1
- net ROT1A: now reaches U1.5 (GP3)
- net ROT1A: now also C10.2, R6.1
- net at C4.1, U4.5: now also C3.1, TP9.1
- net at RV2.2: now also C16.1, TP6.1; no longer U4.3 (+)
- net RotA renamed ROT3A
- net ROT3A: now also C1.1, R9.2
- net RotB renamed ROT3B
- net ROT3B: now also C14.2, R10.1
- new net: R3.1, RV1.1, TP13.1
- new net: J3.1 (Pin_1), R10.2, R_Pullup6.1, TP14.1
- new net: J4.5 (Pin_5), R5.1, R_Pullup1.1, TP18.1
- new net: C15.2, U3.3 (+)
- new net: R4.2, RV2.1, TP12.1
- new net: J4.1 (Pin_1), R6.2, R_Pullup2.1, TP19.1
- new net: J5.5 (Pin_5), R7.1, R_Pullup4.1, TP16.1
- new net: J5.1 (Pin_1), R8.2, R_Pullup5.1, TP17.1
- new net: C16.2, U4.3 (+)
- new net: J3.5 (Pin_5), R9.1, R_Pullup7.1, TP15.1
- new net ROT1B: C9.1, R5.2, U1.4 (GP2)
- new net ROT2A: C2.1, R7.2, U1.9 (GP6)
- no-connect marks 22 -> 20
Other:
- moved on the sheet: J2, LS2, R2, R_Pullup3, Rpullup1, Rpullup2, SW1, U1, U2
